File: EDA/main/CANSAT-M2-2026.kicad_pcb (KiCad board)
At the start: 6 copper layers, 191 parts, among them J1 12402012E212A, J10 2328702-8, J11 532610871, J12 SIM800L V2, J2 1-2328702-0, J3 MSD-4-A, J4 STM32H7_SWD, J5 STM32L0_SWD, J6 SKRPACE010, J7 SKRPACE010, J8 Power, J9 XT30 Battery, U1 TPS63060DSCT, U10 TPS25730DREFR, U11 STM32L031G6U6, U12 TPS22919DCKR, U13 TPS22919DCKR, U14 TPS63060DSCT, U2 ICM-42688-P, U3 MMC5983MA, U4 TMP121AIDBVR, U5 TPS22919DCKR, U6 BMP581, U7 STM32H7S3L8H6, U8 IS42S16800F-7TL, U9 BQ25895RTWT, Y1 ABS07-32.768KHZ-T, Y2 25MHz, Y3 ABS07-32.768KHZ-T

Commit message: Uploaded work
Parts:
- removed R27, R28: 4.7kΩ, Resistor_SMD:R_0402_1005Metric
- added FB1: FerriteBead, Inductor_SMD:L_0603_1608Metric, F.Cu at (246.0, 122.2)
- C16, C17, C31, C32, C33, C34, C35, C36, C37, C38, C39, C40, C41, C42, C43, C44, C45, C46, C47, C48, C49, C50, C51, C52, C53, C54, C55, C56, C57, C58, C59, C60, C61, C62, C63, C64, C65, C66, C67, C68, C69, C7, C70, C71, C72, C73, C74, C75, C76, C77, C78, C79, C80, C81, C82, U8: moved to B.Cu
- moved C114 141.8 mm to (250.3, 156.2), turned to -90 degrees
- moved C113 140.6 mm to (247.6, 156.2), turned to -90 degrees
- moved C112 136.8 mm to (241.7, 156.2), turned to -90 degrees
- moved Y2 128.4 mm to (281.4, 124.4)
- moved U13 127.8 mm to (244.8, 156.1)
- moved Y3 125.9 mm to (272.3, 141.6)
- moved R29 124.7 mm to (280.3, 134.2)
- moved J9 117.8 mm to (30.6, 31.3)
- moved J6 115.7 mm to (279.6, 131.1)
- moved J8 115.6 mm to (50.1, 50.1), turned to 180 degrees
- moved C85 113.5 mm to (276.3, 139.0)
- moved C86 113.5 mm to (276.3, 141.0)
- moved C83 113.0 mm to (280.7, 118.8)
- moved C84 113.0 mm to (280.7, 120.8)
- moved R24 112.9 mm to (41.8, 56.1), turned to -90 degrees
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Connections:
- C10 pad 2: Net-(J3-VDD) -> /3V3
- C106 pad 1: GND -> /3V3
- C107 pad 1: GND -> /3V3
- C108 pad 1: GND -> /3V3
- C109 pad 1: GND -> /3V3
- C11 pad 2: Net-(J3-VDD) -> /3V3
- C112 pad 1: GND -> /3V3
- C2 pad 1: GND -> /3V3
- C23 pad 2: GND -> /3V3
- C27 pad 1: GND -> /3V3
- C28 pad 2: GND -> /3V3
- C29 pad 2: GND -> /3V3
- C3 pad 1: GND -> /3V3
- C30 pad 1: GND -> /3V3
- C31 pad 1: GND -> /3V3
- C32 pad 1: GND -> /3V3
- C33 pad 1: GND -> /3V3
- C34 pad 1: GND -> /3V3
- C35 pad 1: GND -> /3V3
- C36 pad 1: GND -> /3V3
- C37 pad 1: GND -> /3V3
- C38 pad 1: GND -> /3V3
- C39 pad 1: GND -> /3V3
- C4 pad 1: GND -> /3V3
- C40 pad 1: GND -> /3V3
- C41 pad 1: GND -> /3V3
- C42 pad 2: GND -> /3V3
- C43 pad 2: GND -> /3V3
- C44 pad 2: GND -> /3V3
- C45 pad 2: GND -> /3V3
- C46 pad 2: GND -> /3V3
- C47 pad 2: GND -> /3V3
- C48 pad 2: GND -> /3V3
- C49 pad 2: GND -> /3V3
- C5 pad 2: GND -> /3V3
- C50 pad 2: GND -> /3V3
- C51 pad 2: GND -> /3V3
- C52 pad 2: GND -> /3V3
- C53 pad 2: GND -> /3V3
- C54 pad 2: GND -> /3V3
- C55 pad 2: GND -> /3V3
- C56 pad 2: GND -> /3V3
- C57 pad 2: GND -> /3V3
- C58 pad 2: GND -> /3V3
- C59 pad 2: GND -> /3V3
- C6 pad 1: GND -> /3V3
- C60 pad 1: GND -> /3V3
- C61 pad 2: Net-(U7C-DVDD) -> /3V3
- C62 pad 1: GND -> /3V3
- C63 pad 1: GND -> /3V3
- C64 pad 1: GND -> /3V3
- C65 pad 1: GND -> /3V3
- C7 pad 2: GND -> /3V3
- C70 pad 2: Net-(U7C-DVDD) -> /3V3
- C71 pad 2: GND -> /3V3
- C72 pad 2: GND -> /3V3
- C73 pad 2: GND -> /3V3
- C74 pad 2: GND -> /3V3
- C75 pad 2: GND -> /3V3
- C76 pad 2: GND -> /3V3
- C77 pad 1: GND -> /3V3
- C78 pad 1: GND -> /3V3
- C8 pad 2: GND -> /3V3
- C9 pad 2: Net-(J3-VDD) -> /3V3
- C93 pad 1: GND -> /3V3
- C94 pad 1: GND -> /3V3
- C95 pad 1: GND -> /3V3
- C96 pad 1: GND -> /3V3
- C97 pad 1: GND -> /3V3
- J12 pad 3: GND -> /3V3
- J2 pad 2: GND -> /3V3
- J3 pad 4: Net-(J3-VDD) -> /3V3
- J4 pad 1: GND -> /3V3
- J5 pad 1: GND -> /3V3
- J6 pad 2: GND -> /3V3
- J7 pad 2: GND -> /3V3
- R11 pad 1: GND -> /3V3
- R12 pad 1: GND -> /3V3
- R21 pad 2: GND -> /3V3
- R22 pad 2: GND -> /3V3
- R23 pad 2: GND -> /3V3
- R24 pad 2: GND -> /3V3
- R26 pad 2: GND -> /3V3
- R31 pad 1: GND -> /3V3
- R6 pad 1: GND -> /3V3
- R7 pad 1: GND -> /3V3
- R8 pad 1: GND -> /3V3
- R9 pad 1: GND -> /3V3
- U1 pad 9: GND -> /3V3
- U10 pad 38: GND -> /3V3
- U11 pad 1: GND -> /3V3
- U11 pad 17: GND -> /3V3
- U11 pad 5: GND -> /3V3
- U12 pad 1: GND -> /3V3
- U13 pad 1: GND -> /3V3
- U2 pad 10: GND -> /3V3
- U2 pad 5: GND -> /3V3
- U2 pad 8: GND -> /3V3
- U3 pad 13: GND -> /3V3
- U3 pad 2: GND -> /3V3
- U4 pad 3: GND -> /3V3
- U5 pad 1: GND -> /3V3
- U5 pad 5: GND -> /3V3
- U5 pad 6: GND -> /3V3
- U6 pad 1: GND -> /3V3
- U6 pad 10: GND -> /3V3
- U7 pad C1: Net-(U7C-DVDD) -> /3V3
- U7 pad D8: Net-(U7C-DVDD) -> /3V3
- U7 pad D9: GND -> /3V3
- U7 pad F10: GND -> /3V3
- U7 pad F7: GND -> /3V3
- U7 pad F8: GND -> /3V3
- U7 pad F9: GND -> /3V3
- U7 pad G6: GND -> /3V3
- U7 pad G7: GND -> /3V3
- U7 pad G9: GND -> /3V3
- U7 pad H10: GND -> /3V3
- U7 pad H12: GND -> /3V3
- U7 pad H6: GND -> /3V3
- U7 pad J11: GND -> /3V3
- U7 pad J7: GND -> /3V3
- U7 pad J9: GND -> /3V3
- U7 pad K10: GND -> /3V3
- U7 pad K12: GND -> /3V3
- U7 pad K6: GND -> /3V3
- U7 pad K8: GND -> /3V3
- U7 pad L10: GND -> /3V3
- U7 pad L8: GND -> /3V3
- U7 pad L9: GND -> /3V3
- U7 pad M10: GND -> /3V3
- U8 pad 1: GND -> /3V3
- U8 pad 14: GND -> /3V3
- U8 pad 27: GND -> /3V3
- U8 pad 3: GND -> /3V3
- U8 pad 43: GND -> /3V3
- U8 pad 49: GND -> /3V3
- U8 pad 9: GND -> /3V3
Routing:
- net /3V3: track 0.00 -> 119.3 mm, vias 0 -> 7
- net VBUS: track 0.00 -> 23.9 mm
- net CC2: track 0.00 -> 18.6 mm, vias 0 -> 2
- net CC1: track 0.00 -> 18.2 mm, vias 0 -> 2
- net /Power/SYS: track 0.00 -> 15.1 mm
- net /5V: track 0.00 -> 9.44 mm
- net /Power/PPHV: track 0.00 -> 6.53 mm
- net /Interface/3V3_GNSS: track 0.00 -> 6.00 mm
- net /Sensors/3V3_EXT: track 0.00 -> 6.00 mm
- net Net-(U14-FB): track 0.00 -> 5.35 mm
- net Net-(U1-FB): track 0.00 -> 5.25 mm
- net GND: track 0.00 -> 3.84 mm
- net Net-(U1-VAUX): track 0.00 -> 2.71 mm
- net Net-(U14-VAUX): track 0.00 -> 2.49 mm
- net D+: track 0.00 -> 2.48 mm
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
Commit message: Worked on SDRAM
Parts:
- moved C73 54.8 mm to (233.2, 53.5), turned to 0 degrees
- moved C71 53.4 mm to (235.3, 53.9), turned to -90 degrees
- moved C72 53.3 mm to (233.2, 54.3), turned to 0 degrees
- moved U7 52.9 mm to (219.7, 56.2), turned to 180 degrees
- moved C56 52.6 mm to (235.0, 54.3), turned to 180 degrees
- moved C76 52.6 mm to (231.6, 55.1), turned to 0 degrees
- moved C59 51.6 mm to (233.2, 55.2), turned to 0 degrees
- moved C55 51.1 mm to (234.8, 55.1), turned to 0 degrees
- moved C54 50.7 mm to (236.4, 55.1), turned to 0 degrees
- moved C75 50.5 mm to (232.3, 55.9), turned to 0 degrees
- moved C74 49.4 mm to (231.6, 56.7), turned to 0 degrees
- moved C58 48.6 mm to (233.2, 56.7), turned to 0 degrees
- moved C53 47.3 mm to (237.3, 56.7), turned to 180 degrees
- moved C52 45.8 mm to (237.4, 57.5), turned to 180 degrees
- moved C57 45.5 mm to (233.2, 58.3), turned to 0 degrees
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Routing:
- net Net-(U7C-VCAP4): vias 0 -> 1
- net Net-(U7C-VCAP3): vias 0 -> 1
- net Net-(U7C-VCAP2): vias 0 -> 1
- net Net-(U7C-VCAP1): vias 0 -> 1
- net GND: vias 0 -> 40
- net /VDDA: vias 0 -> 2
- net /ToF_XSHUT: vias 0 -> 1
- net /ToF_SDA: vias 0 -> 1
- net /ToF_SCL: vias 0 -> 1
- net /ToF_INT: vias 0 -> 1
- net /SWDIO: vias 0 -> 1
- net /SWCLK: vias 0 -> 1
- net /SPI_CS_TMP_OUT: vias 0 -> 1
- net /SPI_CS_TMP_IN: vias 0 -> 1
- net /SPI_CS_PWR-MCU: vias 0 -> 1
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- added copper zone on In3.Cu, net /3V3
- added copper zone on In1.Cu, net GND
- added copper zone on In4.Cu, net GND

Commit message: Uploaded work
Parts:
- removed C31, C32, C38, C40, C42, C44, C46: 100nF, Capacitor_SMD:C_0402_1005Metric
- removed C33, C34, C39, C41, C43, C45, C47: 10nF, Capacitor_SMD:C_0402_1005Metric
- removed C35, C49: 4.7uF, Capacitor_SMD:C_0603_1608Metric
- removed C36, C50: 1uF, Capacitor_SMD:C_0603_1608Metric
- removed C37, C48: 10uF, Capacitor_SMD:C_0603_1608Metric
- removed U8: IS42S16800F-7TL, CANSAT-lib:TSOP-II-54_ISI
- added L1: 1uH, Inductor_SMD:L_1008_2520Metric, B.Cu at (230.7, 58.7)
- added L2: 2.2uH, Inductor_SMD:L_Wuerth_MAPI-4020, F.Cu at (225.2, 53.4)
- added L3: 1uH, Inductor_SMD:L_1008_2520Metric, B.Cu at (222.5, 114.4)
- added REF**: MountingHole_2.7mm_M2.5_DIN965_Pad, MountingHole:MountingHole_2.7mm_M2.5_DIN965_Pad, F.Cu at (255.7, 132.2)
- added REF**: MountingHole_2.7mm_M2.5_DIN965_Pad, MountingHole:MountingHole_2.7mm_M2.5_DIN965_Pad, F.Cu at (255.8, 37.5)
- added REF**: MountingHole_2.7mm_M2.5_DIN965_Pad, MountingHole:MountingHole_2.7mm_M2.5_DIN965_Pad, F.Cu at (206.1, 132.2)
- added REF**: MountingHole_2.7mm_M2.5_DIN965_Pad, MountingHole:MountingHole_2.7mm_M2.5_DIN965_Pad, F.Cu at (206.6, 37.5)
- C10, C11, C115, C116, C117, C118, C119, C120, C121, C122, C123, C124, C125, C126, C25, C26, C27, C28, C29, C30, C87, C88, C89, C9, C90, C91, C92, C93, C94, C95, C96, C97, C98, J3, J7, R1, R11, R12, R2, R3, R30, R31, R32, R33, R34, R4, R5, R6, R7, R8, R9, U1, U11, U14, Y1: moved to B.Cu
- J12: footprint CANSAT-lib:PinHeader_1x07_P2.54mm_Vertical -> CANSAT-lib:AMPHENOL_91601-307LF; moved to B.Cu
- moved C102 203.4 mm to (237.2, 52.3), turned to 90 degrees
- moved C101 200.7 mm to (234.7, 52.3), turned to 90 degrees
- moved C24 197.5 mm to (223.6, 63.4), turned to 90 degrees
- moved C22 189.5 mm to (250.4, 60.4)
- moved C12 188.7 mm to (249.3, 47.1)
- moved C17 188.7 mm to (246.3, 44.1)
- moved C19 188.7 mm to (253.2, 52.2)
- moved C20 188.7 mm to (254.7, 52.2)
- moved R18 188.7 mm to (244.2, 56.0)
- moved R21 188.7 mm to (251.8, 58.0)
- moved R22 188.7 mm to (251.8, 56.9)
- moved U10 188.7 mm to (247.7, 54.9)
- moved C13 188.7 mm to (248.1, 47.1)
- moved C14 188.7 mm to (246.9, 47.1)
- moved C15 188.7 mm to (245.6, 47.7)
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Connections:
- J1 pad A6: D+ -> /USB-DP
- J1 pad A7: D- -> /USB-DM
- J1 pad B6: D+ -> /USB-DP
- J1 pad B7: D- -> /USB-DM
- U7 pad A13: /FMC_CS -> unconnected-(U7B-PE14-PadA13)
- U7 pad A2: /FMC_D9 -> unconnected-(U7B-PE0-PadA2)
- U7 pad A3: /FMC_A11 -> unconnected-(U7B-PF3-PadA3)
- U7 pad A4: /FMC_A10 -> unconnected-(U7B-PF2-PadA4)
- U7 pad A7: unconnected-(U7B-PM12-PadA7) -> /USB-DM
- U7 pad B12: /FMC_CAS -> unconnected-(U7B-PE13-PadB12)
- U7 pad B13: /FMC_A7 -> unconnected-(U7A-PD1-PadB13)
- U7 pad B2: /FMC_D11 -> unconnected-(U7B-PE2-PadB2)
- U7 pad B5: /FMC_A8 -> unconnected-(U7B-PF0-PadB5)
- U7 pad B6: /FMC_D8 -> unconnected-(U7A-PD7-PadB6)
- U7 pad B7: unconnected-(U7B-PM11-PadB7) -> /USB-DP
- U7 pad C12: /FMC_WE -> unconnected-(U7B-PE11-PadC12)
- U7 pad C13: /FMC_A6 -> unconnected-(U7A-PD0-PadC13)
- U7 pad C14: /FMC_D0 -> unconnected-(U7A-PA12-PadC14)
- U7 pad C15: /FMC_D1 -> unconnected-(U7A-PA11-PadC15)
- U7 pad C3: /FMC_D10 -> unconnected-(U7B-PE1-PadC3)
- U7 pad C5: /FMC_A9 -> unconnected-(U7B-PF1-PadC5)
- U7 pad D11: /FMC_CKE -> unconnected-(U7B-PE15-PadD11)
- U7 pad D14: /FMC_D3 -> unconnected-(U7A-PA9-PadD14)
- U7 pad E1: /FMC_D15 -> unconnected-(U7B-PE6-PadE1)
- U7 pad E11: /FMC_RAS -> unconnected-(U7B-PE12-PadE11)
- U7 pad E13: /FMC_D2 -> unconnected-(U7A-PA10-PadE13)
- U7 pad E2: /FMC_D13 -> unconnected-(U7B-PE4-PadE2)
- U7 pad F12: /FMC_D4 -> unconnected-(U7A-PA8-PadF12)
- U7 pad F14: /FMC_NBL0 -> unconnected-(U7B-PN1-PadF14)
- U7 pad F4: /FMC_D14 -> unconnected-(U7B-PE5-PadF4)
- U7 pad F5: /FMC_D12 -> unconnected-(U7B-PE3-PadF5)
- U7 pad G15: /FMC_D7 -> unconnected-(U7B-PN11-PadG15)
- U7 pad H13: /FMC_D6 -> unconnected-(U7B-PN10-PadH13)
- U7 pad H14: /FMC_D5 -> unconnected-(U7B-PN9-PadH14)
- U7 pad J14: /FMC_CLK -> unconnected-(U7B-PN6-PadJ14)
- U7 pad K3: /FMC_NBL1 -> unconnected-(U7A-PC0-PadK3)
- U7 pad L1: /FMC_A0 -> unconnected-(U7A-PC1-PadL1)
- U7 pad L2: /FMC_A1 -> unconnected-(U7A-PC2-PadL2)
- U7 pad L3: /FMC_A2 -> unconnected-(U7A-PC3-PadL3)
- U7 pad L5: /FMC_A3 -> unconnected-(U7A-PC4-PadL5)
- U7 pad M6: /FMC_A4 -> unconnected-(U7B-PE7-PadM6)
- U7 pad N3: /FMC_A5 -> unconnected-(U7A-PC5-PadN3)
- U7 pad P5: /FMC_BA0 -> unconnected-(U7B-PE9-PadP5)
- U7 pad R2: unconnected-(U7A-PB1-PadR2) -> /GNSS_PPS
- U7 pad R5: /FMC_BA1 -> unconnected-(U7B-PE10-PadR5)
Routing:
- net /3V3: track 119.3 -> 53.9 mm, vias 31 -> 30
- net /Power/PPHV: track 6.53 -> 57.5 mm, vias 0 -> 5
- net /Power/LDO_3V3: track 0.00 -> 23.4 mm, vias 0 -> 5
- net Net-(C105-Pad1): track 0.00 -> 20.6 mm
- net /Power/PWR_SDA: track 2.08 -> 18.7 mm, vias 0 -> 1
- net /Power/PWR_SCL: track 1.80 -> 17.6 mm, vias 0 -> 1
- net Net-(U9-BAT_13): track 0.00 -> 13.5 mm
- net /Power/NRST: track 0.00 -> 11.6 mm, vias 0 -> 1
- net /Power/SWCLK: track 0.00 -> 11.4 mm, vias 0 -> 1
- net /Power/ADCIN4: track 0.00 -> 10.5 mm
- net /Power/OSC_OUT: track 0.00 -> 9.77 mm
- net /Power/OSC_IN: track 0.00 -> 9.41 mm
- net /Power/SYS: track 15.1 -> 24.2 mm, vias 0 -> 4
- net /Power/ADCIN3: track 0.00 -> 8.64 mm
- net /Power/SWDIO: track 0.00 -> 7.18 mm, vias 0 -> 1
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Other:
- board outline added: 55 x 100 mm

Commit message: PCB done
Parts:
- removed C115, C126: 22uF, Capacitor_SMD:C_0603_1608Metric
- removed C116, C125: 10uF, Capacitor_SMD:C_0603_1608Metric
- removed C117, C124, C60: 4.7uF, Capacitor_SMD:C_0603_1608Metric
- removed C118, C123: 1uF, Capacitor_SMD:C_0603_1608Metric
- removed C119, C120, C122: 100nF, Capacitor_SMD:C_0402_1005Metric
- removed C121: 10pF, Capacitor_SMD:C_0402_1005Metric
- removed J12: SIM800L V2, CANSAT-lib:AMPHENOL_91601-307LF
- removed L3: 1uH, Inductor_SMD:L_1008_2520Metric
- removed R33: 1.8MΩ, Resistor_SMD:R_0402_1005Metric
- removed R34: 200kΩ, Resistor_SMD:R_0402_1005Metric
- removed U14: TPS63060DSCT, CANSAT-lib:CONV_TPS63060DSCT
- added R27: 10kΩ, Resistor_SMD:R_0402_1005Metric, F.Cu at (133.0, 60.4)
- added R28: 10kΩ, Resistor_SMD:R_0402_1005Metric, F.Cu at (134.4, 58.9)
- C109, C110, C111, C3, C4, FB1, U12, U2: moved to B.Cu
- moved C86 181.5 mm to (108.8, 71.2)
- moved C85 177.2 mm to (113.3, 69.6), turned to -90 degrees
- moved C84 177.2 mm to (109.0, 77.0)
- moved Y2 176.5 mm to (111.1, 77.7), turned to -90 degrees
- moved Y3 174.8 mm to (112.0, 71.9)
- moved C83 174.0 mm to (111.2, 79.6)
- moved C80 171.8 mm to (111.2, 83.4), turned to -90 degrees
- moved C82 169.7 mm to (113.4, 80.7), turned to -90 degrees
- moved C70 164.7 mm to (115.0, 72.2), turned to -90 degrees
- moved C64 164.4 mm to (110.9, 74.6), turned to 90 degrees
- moved R29 163.2 mm to (131.9, 66.4), turned to -90 degrees
- moved C81 161.7 mm to (115.5, 80.1), turned to -90 degrees
- moved C62 160.7 mm to (114.3, 77.6), turned to 90 degrees
- moved C77 159.4 mm to (123.6, 85.1)
- moved C78 159.4 mm to (123.6, 86.6)
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Connections:
- net Net-(U9-REGN) renamed /Power/REGN
- C107 pad 1: /3V3 -> /Sensors/SENS_3V3
- C108 pad 1: /3V3 -> /Sensors/SENS_3V3
- C2 pad 1: /3V3 -> /Sensors/SENS_3V3
- C3 pad 1: /3V3 -> /Sensors/SENS_3V3
- C4 pad 1: /3V3 -> /Sensors/SENS_3V3
- C5 pad 2: /3V3 -> /Sensors/SENS_3V3
- C6 pad 1: /3V3 -> /Sensors/SENS_3V3
- C8 pad 2: /3V3 -> /Sensors/SENS_3V3
- R26 pad 1: BAT_INT -> /Power/BQ_INT
- RF1 pad 1: unconnected-(RF1-GND-Pad1) -> GND
- RF1 pad 10: unconnected-(RF1-GND-Pad10) -> GND
- RF1 pad 2: unconnected-(RF1-VCC-Pad2) -> /3V3
- RF1 pad 3: unconnected-(RF1-EN-Pad3) -> /RF_EN
- RF1 pad 4: unconnected-(RF1-CPS-Pad4) -> /RF_CPS
- RF1 pad 5: unconnected-(RF1-CS-Pad5) -> /SPI5_RF_CS
- RF1 pad 6: unconnected-(RF1-SDI-Pad6) -> /SPI5_SDO
- RF1 pad 7: unconnected-(RF1-SDO-Pad7) -> /SPI5_SDI
- RF1 pad 8: unconnected-(RF1-CLK-Pad8) -> /SPI5_CLK
- RF1 pad 9: unconnected-(RF1-INTn-Pad9) -> /RF_INT
- U11 pad 23: unconnected-(U11A-PA15-Pad23) -> /Power/BQ_INT
- U2 pad 10: /3V3 -> /Sensors/SENS_3V3
- U2 pad 5: /3V3 -> /Sensors/SENS_3V3
- U2 pad 8: /3V3 -> /Sensors/SENS_3V3
- U3 pad 13: /3V3 -> /Sensors/SENS_3V3
- U3 pad 2: /3V3 -> /Sensors/SENS_3V3
- U4 pad 3: /3V3 -> /Sensors/SENS_3V3
- U5 pad 5: /3V3 -> /Sensors/SENS_3V3
- U5 pad 6: /3V3 -> /Sensors/SENS_3V3
- U6 pad 1: /3V3 -> /Sensors/SENS_3V3
- U6 pad 10: /3V3 -> /Sensors/SENS_3V3
- U7 pad C7: unconnected-(U7B-PM13-PadC7) -> /SPI5_SDO
- U7 pad C8: unconnected-(U7B-PM14-PadC8) -> /SPI5_SDI
- U7 pad D7: /MCU>SIM_TX -> unconnected-(U7A-PD5-PadD7)
- U7 pad E4: /5V_EN -> unconnected-(U7A-PC13-PadE4)
- U7 pad E7: /MCU<SIM_RX -> unconnected-(U7A-PD6-PadE7)
- U7 pad H4: unconnected-(U7B-PF7-PadH4) -> /SPI5_CLK
- U7 pad N12: /ONB_SENS_EN -> unconnected-(U7B-PO0-PadN12)
- U7 pad N3: unconnected-(U7A-PC5-PadN3) -> /GNSS_EN
- U7 pad P3: unconnected-(U7B-PF13-PadP3) -> /GNSS_RST
- U7 pad P4: unconnected-(U7B-PF14-PadP4) -> /RF_INT
- U7 pad R14: unconnected-(U7A-PD10-PadR14) -> /ONB_SENS_EN
- U7 pad R5: unconnected-(U7B-PE10-PadR5) -> /SPI5_RF_CS
- U7 pad R8: unconnected-(U7B-PP4-PadR8) -> /RF_CPS
- U7 pad R9: unconnected-(U7B-PO5-PadR9) -> /RF_EN
- U9 pad 7: BAT_INT -> /Power/BQ_INT
Routing:
- net /Sensors/SENS_3V3: track 0.00 -> 117.1 mm, vias 0 -> 8
- net /SPI2_SCK: track 0.00 -> 99.1 mm, vias 1 -> 0
- net /SPI2_MISO: track 0.00 -> 79.5 mm, vias 1 -> 0
- net Net-(J3-DAT1): track 0.00 -> 64.4 mm
- net /SPI2_MOSI: track 0.00 -> 64.4 mm, vias 1 -> 3
- net Net-(J3-CMD): track 0.00 -> 64.3 mm
- net Net-(J3-DAT0): track 0.00 -> 64.2 mm
- net Net-(J3-DAT2): track 0.00 -> 63.9 mm
- net Net-(J3-CD/DAT3): track 0.00 -> 63.7 mm
- net /SDMMC_CD: track 0.00 -> 62.4 mm
- net /SDMMC_CK: track 0.00 -> 62.4 mm
- net /SPI_CS_TMP_IN: track 0.00 -> 60.3 mm, vias 1 -> 6
- net /NRST: track 0.00 -> 58.2 mm, vias 1 -> 2
- net /BAR_INT: track 0.00 -> 55.6 mm, vias 1 -> 2
- net /SPI_CS_BAR: track 0.00 -> 54.7 mm, vias 1 -> 2
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- added copper zone on In2.Cu, net /3V3
- added copper zone on B.Cu, net GND
- added copper zone on F.Cu, net GND
- removed copper zone on In3.Cu, net /3V3
- removed copper zone on In4.Cu, net GND
Other:
- outline, holes or cut-outs redrawn
- copper layers 6 -> 4
