File: EDA/main/CANSAT-M2-2026.kicad_sch (KiCad schematic)
At the start: 44 parts, among them J4 STM32H7_SWD, J6 SKRPACE010, U7 STM32H7S3L8H6, Y2 25MHz, Y3 ABS07-32.768KHZ-T

Commit message: PCB done
Parts:
- removed C60: 4.7uF, Capacitor_SMD:C_0603_1608Metric, symbol Device:C
- C51, C52, C53, C54, C55, C56, C57, C58, C59, C61, C63, C65, C7, C71, C72, C73, C74, C75, C76, C79, C81: Manufacturer Part (none) -> CL05B104KP5NNNC
- C62, C70, C78: Manufacturer Part (none) -> CL10A475KP8NNNC
- C64, C77, C80, C82: Manufacturer Part (none) -> CL10B105MO8NNWC
- C66, C67, C68, C69: Manufacturer Part (none) -> CL10A225KO8NNNC
- C83, C84: Manufacturer Part (none) -> CL05C100JB5NNNC
- C85, C86: Manufacturer Part (none) -> CL05C180JB5NNNC
- J6: Manufacturer Part (none) -> SKRPACE010
- R29: Manufacturer Part (none) -> RC0402FR-0710KL
- U7: Manufacturer Part (none) -> STM32H7S3L8H6H
- Y2: Manufacturer Part (none) -> ECS-160-9-37-CKM-TR
- Y3: Manufacturer Part (none) -> ABS07-32.768KHZ-T
Connections:
- net GNSS_EN: now also U7.N3 (PC5)
- net GNSS_RST: now also U7.P3 (PF13)
- net ONB_SENS_EN: now also U7.R14 (PD10); no longer U7.N12 (PO0)
- net SPI5_SDO: now reaches U7.C7 (PM13)
- net SPI5_SDI: now reaches U7.C8 (PM14)
- net SPI5_CLK: now reaches U7.H4 (PF7)
- net RF_INT: now reaches U7.P4 (PF14)
- net SPI5_RF_CS: now reaches U7.R5 (PE10)
- net RF_CPS: now reaches U7.R8 (PP4)
- net RF_EN: now reaches U7.R9 (PO5)
- net 5V_EN: no longer names the net of U7.E4 (PC13)
- net MCU<SIM_RX: no longer names the net of U7.E7 (PD6)
- net MCU>SIM_TX: no longer names the net of U7.D7 (PD5)
Other:
- sheet Interface ports: added RF_CPS, RF_EN, RF_INTn, SPI5_CLK, SPI5_RF_CS, SPI5_SDI, SPI5_SDO; removed 5V, SIM_RST, SIM_RX, SIM_TX
- sheet Power ports: added none; removed 5V_EN
