File: EDA/main/Interface.kicad_sch (KiCad schematic)
At the start: 23 parts, among them J1 12402012E212A, J11 532610871, J12 SIM800L V2, J3 MSD-4-A, U13 TPS22919DCKR

Commit message: Uploaded work
Connections:
- net 3V3: now also C10.2, C11.2, C9.2, J3.4 (VDD); no longer C10.1, C11.1, C9.1
- net COVER_GND: now also C10.1, C11.1, C9.1
Changed lines of the file:
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@@
-	)
-	(junction
-		(at 134.62 81.28)
-		(diameter 0)
-		(color 0 0 0 0)
 	)
 	(junction
@@
 	)
 	(junction
+		(at 134.62 88.9)
+		(diameter 0)
+		(color 0 0 0 0)
+	)
+	(junction
 		(at 128.27 106.68)
 		(diameter 0)
@@
 	(junction
 		(at 201.93 137.16)
+		(diameter 0)
+		(color 0 0 0 0)
+	)
+	(junction
+		(at 148.59 81.28)
 		(diameter 0)
 		(color 0 0 0 0)
@@
 	(wire
 		(pts
-			(xy 133.35 81.28) (xy 134.62 81.28)
-		)
-		(stroke
-			(width 0)
-			(type default)
-		)
-	)
-	(wire
-		(pts
 			(xy 104.14 116.84) (xy 105.41 116.84)
 		)
@@
 	(wire
 		(pts
+			(xy 148.59 81.28) (xy 153.67 81.28)
+		)
+		(stroke
+			(width 0)
+			(type default)
+		)
+	)
+	(wire
+		(pts
 			(xy 135.89 128.27) (xy 143.51 128.27)
 		)
@@
 		(pts
 			(xy 260.35 139.7) (xy 267.97 139.7)
+		)
+		(stroke
+			(width 0)
+			(type default)
+		)
+	)
+	(wire
+		(pts
+			(xy 133.35 88.9) (xy 134.62 88.9)
 		)
 		(stroke
@@
 	(hierarchical_label "3V3"
 		(shape input)
-		(at 133.35 81.28 180)
+		(at 133.35 88.9 180)
 		(effects
 			(font
@@
 					(unit 1)
 				)
+			)
+		)
+	)
+	(symbol
+		(lib_id "power:GND")
+		(at 153.67 81.28 0)
+		(unit 1)
+		(exclude_from_sim no)
+		(in_bom yes)
+		(on_board yes)
+		(dnp no)
+		(fields_autoplaced yes)
+		(property "Reference" "#PWR0110"
+			(at 153.67 87.63 0)
+			(effects
+				(font
+					(size 1.27 1.27)
+				)
+				(hide yes)
+			)
+		)
+		(property "Value" "GND"
+			(at 153.67 86.36 0)
+			(effects
+				(font
+					(size 1.27 1.27)
+				)
+			)
+		)
+		(property "Footprint" ""
+			(at 153.67 81.28 0)
+			(effects
+				(font
+					(size 1.27 1.27)
+				)
+				(hide yes)
+			)
+		)
+		(property "Datasheet" ""
+			(at 153.67 81.28 0)
+			(effects
+				(font
+					(size 1.27 1.27)
+				)
+				(hide yes)
+			)
+		)
+		(property "Description" "Power symbol creates a global label with name \"GND\" , ground"
+			(at 153.67 81.28 0)
+			(effects
+				(font
+					(size 1.27 1.27)
+				)
+				(hide yes)
+			)
+		)
+		(pin "1"
+		)
+		(instances
+			(project "CANSAT-M2-2026"
+				(path "/7307961f-7cb3-4b36-8f89-29751d54bb23/b4d81b11-a1a2-498b-bd71-8ef439ae7231"
+					(reference "#PWR0110")
+					(unit 1)
+				)

Commit message: Uploaded work
Parts:
- J12: footprint CANSAT-lib:PinHeader_1x07_P2.54mm_Vertical -> CANSAT-lib:AMPHENOL_91601-307LF
Connections:
- net D+ renamed USB-DP
- net D- renamed USB-DM
Changed lines of the file:
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@@
-		)
-	)
-	(global_label "D-"
-		(shape bidirectional)
-		(at 153.67 45.72 180)
-		(fields_autoplaced yes)
-		(effects
-			(font
-				(size 1.27 1.27)
-			)
-			(justify right)
-		)
-		(property "Intersheetrefs" "${INTERSHEET_REFS}"
-			(at 146.7311 45.72 0)
-			(effects
-				(font
-					(size 1.27 1.27)
-				)
-				(justify right)
-				(hide yes)
-			)
-		)
-	)
-	(global_label "D+"
-		(shape bidirectional)
-		(at 189.23 48.26 0)
-		(fields_autoplaced yes)
-		(effects
-			(font
-				(size 1.27 1.27)
-			)
-			(justify left)
-		)
-		(property "Intersheetrefs" "${INTERSHEET_REFS}"
-			(at 196.1689 48.26 0)
-			(effects
-				(font
-					(size 1.27 1.27)
-				)
-				(justify left)
-				(hide yes)
-			)
 		)
 	)
@@
 		)
 	)
-	(global_label "D-"
-		(shape bidirectional)
-		(at 189.23 45.72 0)
-		(fields_autoplaced yes)
-		(effects
-			(font
-				(size 1.27 1.27)
-			)
-			(justify left)
-		)
-		(property "Intersheetrefs" "${INTERSHEET_REFS}"
-			(at 196.1689 45.72 0)
-			(effects
-				(font
-					(size 1.27 1.27)
-				)
-				(justify left)
-				(hide yes)
-			)
-		)
-	)
 	(global_label "CC2"
 		(shape bidirectional)
@@
 		)
 	)
-	(global_label "D+"
-		(shape bidirectional)
-		(at 153.67 43.18 180)
-		(fields_autoplaced yes)
-		(effects
-			(font
-				(size 1.27 1.27)
-			)
-			(justify right)
-		)
-		(property "Intersheetrefs" "${INTERSHEET_REFS}"
-			(at 146.7311 43.18 0)
-			(effects
-				(font
-					(size 1.27 1.27)
-				)
-				(justify right)
-				(hide yes)
-			)
-		)
-	)
 	(hierarchical_label "GNSS_TX"
 		(shape output)
@@
 		)
 	)
+	(hierarchical_label "USB-DP"
+		(shape bidirectional)
+		(at 189.23 48.26 0)
+		(effects
+			(font
+				(size 1.27 1.27)
+			)
+			(justify left)
+		)
+	)
+	(hierarchical_label "USB-DM"
+		(shape bidirectional)
+		(at 153.67 45.72 180)
+		(effects
+			(font
+				(size 1.27 1.27)
+			)
+			(justify right)
+		)
+	)
 	(hierarchical_label "SDMMC_D0"
 		(shape bidirectional)
 		(at 104.14 104.14 180)
+		(effects
+			(font
+				(size 1.27 1.27)
+			)
+			(justify right)
+		)
+	)
+	(hierarchical_label "USB-DM"
+		(shape bidirectional)
+		(at 189.23 45.72 0)
+		(effects
+			(font
+				(size 1.27 1.27)
+			)
+			(justify left)
+		)
+	)
+	(hierarchical_label "USB-DP"
+		(shape bidirectional)
+		(at 153.67 43.18 180)
 		(effects
 			(font
@@
 	)
 	(symbol
+		(lib_id "CANSAT-lib:Conn_01x07_Pin")
+		(at 147.32 152.4 0)
+		(mirror y)
+		(unit 1)
+		(exclude_from_sim no)
+		(in_bom yes)
+		(on_board yes)
+		(dnp no)
+		(property "Reference" "J12"
+			(at 139.7 140.208 0)
+			(effects
+				(font
+					(size 1.27 1.27)
+				)
+				(justify right)
+			)
+		)
+		(property "Value" "SIM800L V2"
+			(at 136.398 141.986 0)
+			(effects
+				(font
+					(size 1.27 1.27)
+				)
+				(justify right)
+			)
+		)
+		(property "Footprint" "CANSAT-lib:AMPHENOL_91601-307LF"
+			(at 147.32 152.4 0)
+			(effects
+				(font
+					(size 1.27 1.27)
+				)
+				(hide yes)
+			)
+		)
+		(property "Datasheet" "~"
+			(at 147.32 152.4 0)
+			(effects
+				(font
+					(size 1.27 1.27)
+				)
+				(hide yes)
+			)
+		)
+		(property "Description" "Generic connector, single row, 01x07, script generated"
+			(at 147.32 152.4 0)
+			(effects
+				(font
+					(size 1.27 1.27)
+				)
+				(hide yes)
+			)
+		)
+		(pin "1"
+		)
+		(pin "6"
+		)
+		(pin "7"
+		)
+		(pin "5"
+		)
+		(pin "2"
+		)
+		(pin "3"
+		)
+		(pin "4"
+		)
+		(instances
+			(project ""
+				(path "/7307961f-7cb3-4b36-8f89-29751d54bb23/b4d81b11-a1a2-498b-bd71-8ef439ae7231"
+					(reference "J12")
+					(unit 1)
+				)
+			)
+		)
+	)
+	(symbol
 		(lib_id "CANSAT-lib:12402012E212A")
 		(at 171.45 45.72 0)
@@
 					(unit 1)
 				)
-			)
-		)
-	)
-	(symbol
-		(lib_id "CANSAT-lib:Conn_01x07_Pin")
-		(at 147.32 152.4 0)
-		(mirror y)
-		(unit 1)
-		(exclude_from_sim no)
-		(in_bom yes)
-		(on_board yes)
-		(dnp no)
-		(fields_autoplaced yes)
-		(property "Reference" "J12"
-			(at 146.685 139.7 0)
-			(effects
-				(font
-					(size 1.27 1.27)
-				)
-			)
-		)
-		(property "Value" "SIM800L V2"
-			(at 146.685 142.24 0)
-			(effects
-				(font
-					(size 1.27 1.27)
-				)
-			)
-		)
-		(property "Footprint" "CANSAT-lib:PinHeader_1x07_P2.54mm_Vertical"
-			(at 147.32 152.4 0)
-			(effects
-				(font
-					(size 1.27 1.27)
-				)
-				(hide yes)
-			)
-		)
-		(property "Datasheet" "~"
-			(at 147.32 152.4 0)
-			(effects
-				(font
-					(size 1.27 1.27)
-				)
-				(hide yes)
-			)
-		)
-		(property "Description" "Generic connector, single row, 01x07, script generated"
-			(at 147.32 152.4 0)
-			(effects
-				(font
-					(size 1.27 1.27)
-				)
-				(hide yes)
-			)
-		)
-		(pin "4"
-		)
-		(pin "6"
-		)
-		(pin "1"
-		)
-		(pin "7"
-		)
-		(pin "2"
-		)
-		(pin "3"
-		)
-		(pin "5"
-		)
-		(instances
-			(project ""
-				(path "/7307961f-7cb3-4b36-8f89-29751d54bb23/b4d81b11-a1a2-498b-bd71-8ef439ae7231"
-					(reference "J12")
-					(unit 1)
-				)

Commit message: PCB done
Parts:
- removed J12: SIM800L V2, CANSAT-lib:AMPHENOL_91601-307LF, symbol CANSAT-lib:Conn_01x07_Pin
- C10, C112, C114: Manufacturer Part (none) -> CL10B105MO8NNWC
- C11, C113: Manufacturer Part (none) -> CL10X106MO8NRNC
- C9: Manufacturer Part (none) -> CL05B104KP5NNNC
- J1: Manufacturer Part (none) -> 12402012E212A
- J11: Manufacturer Part (none) -> 0532610871
- J3: Manufacturer Part (none) -> MSD-4-A
- R1, R2, R3, R4, R5: Manufacturer Part (none) -> RC0402FR-0722RL
- R11, R12, R6, R7, R8, R9: Manufacturer Part (none) -> RC0402FR-0710KL
- U13: Manufacturer Part (none) -> TPS22919DCKR
Connections:
- net 3V3: now also RF1.2 (VCC)
- net COVER_GND: now also RF1.1 (GND), RF1.10 (GND)
- net RF_EN: now reaches RF1.3 (EN)
- net RF_CPS: now reaches RF1.4 (CPS)
- net SPI5_RF_CS: now reaches RF1.5 (CS)
- net SPI5_SDI: now reaches RF1.6 (SDI)
- net SPI5_SDO: now reaches RF1.7 (SDO)
- net SPI5_CLK: now reaches RF1.8 (CLK)
- net RF_INTn: now reaches RF1.9 (INTn)
