File: EDA/main/Sensors.kicad_sch (KiCad schematic)
At the start: 21 parts, among them J10 2328702-8, J2 1-2328702-0, U12 TPS22919DCKR, U2 ICM-42688-P, U3 MMC5983MA, U4 TMP121AIDBVR, U5 TPS22919DCKR, U6 BMP581

Commit message: PCB done
Parts:
- C1, C107, C110: Manufacturer Part (none) -> CL10X106MO8NRNC
- C106, C108, C109, C111, C2: Manufacturer Part (none) -> CL10B105MO8NNWC
- C3, C4, C5, C6, C8: Manufacturer Part (none) -> CL05B104KP5NNNC
- J10: Manufacturer Part (none) -> 2328702-8
- J2: Manufacturer Part (none) -> 1-2328702-0
- U12, U5: Manufacturer Part (none) -> TPS22919DCKR
- U2: Manufacturer Part (none) -> ICM-42688-P
- U3: Manufacturer Part (none) -> MMC5983MA
- U4: Manufacturer Part (none) -> TMP121AIDBVR
- U6: Manufacturer Part (none) -> BMP581
Connections:
- net 3V3: no longer C107.1, C108.1, C2.1, C3.1, C4.1, C5.2, C6.1, C8.2, U2.10 (RESV), U2.5 (VDDIO), U2.8 (VDD), U3.13 (VDDIO), U3.2 (VDD), U4.3 (V+), U5.5 (QOD), U5.6 (VOUT), U6.1 (VDDIO), U6.10 (VDD)
- new net SENS_3V3: C107.1, C108.1, C2.1, C3.1, C4.1, C5.2, C6.1, C8.2, U2.10 (RESV), U2.5 (VDDIO), U2.8 (VDD), U3.13 (VDDIO), U3.2 (VDD), U4.3 (V+), U5.5 (QOD), U5.6 (VOUT), U6.1 (VDDIO), U6.10 (VDD)
Changed lines of the file:
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@@
 	(wire
 		(pts
-			(xy 266.7 92.71) (xy 270.51 92.71)
+			(xy 266.7 92.71) (xy 276.86 92.71)
 		)
 		(stroke
@@
 	(wire
 		(pts
-			(xy 92.71 134.62) (xy 97.79 134.62)
+			(xy 92.71 134.62) (xy 102.87 134.62)
 		)
 		(stroke
@@
 	(wire
 		(pts
-			(xy 118.11 176.53) (xy 125.73 176.53)
+			(xy 115.57 176.53) (xy 125.73 176.53)
 		)
 		(stroke
@@
 	(wire
 		(pts
-			(xy 189.23 87.63) (xy 194.31 87.63)
+			(xy 184.15 87.63) (xy 194.31 87.63)
 		)
 		(stroke
@@
 	(wire
 		(pts
-			(xy 78.74 175.26) (xy 87.63 175.26)
+			(xy 78.74 175.26) (xy 88.9 175.26)
 		)
 		(stroke
@@
 	(wire
 		(pts
-			(xy 262.89 87.63) (xy 270.51 87.63)
+			(xy 262.89 87.63) (xy 276.86 87.63)
 		)
 		(stroke
@@
 	(wire
 		(pts
-			(xy 26.67 175.26) (xy 35.56 175.26)
+			(xy 25.4 175.26) (xy 35.56 175.26)
 		)
 		(stroke
@@
 		)
 	)
-	(label "3V3"
-		(at 97.79 134.62 180)
+	(label "SENS_3V3"
+		(at 102.87 134.62 180)
 		(effects
 			(font
@@
 		)
 	)
-	(label "3V3"
-		(at 87.63 175.26 180)
+	(label "SENS_3V3"
+		(at 88.9 175.26 180)
 		(effects
 			(font
@@
 		)
 	)
-	(label "3V3"
-		(at 118.11 176.53 0)
+	(label "SENS_3V3"
+		(at 115.57 176.53 0)
 		(effects
 			(font
@@
 		)
 	)
-	(label "3V3"
+	(label "SENS_3V3"
 		(at 185.42 130.81 0)
 		(effects
@@
 		)
 	)
-	(label "3V3"
-		(at 189.23 87.63 0)
+	(label "SENS_3V3"
+		(at 184.15 87.63 0)
 		(effects
 			(font
@@
 		)
 	)
-	(label "3V3"
-		(at 270.51 92.71 180)
+	(label "SENS_3V3"
+		(at 276.86 92.71 180)
 		(effects
 			(font
@@
 		)
 	)
-	(label "3V3"
+	(label "SENS_3V3"
 		(at 261.62 135.89 180)
 		(effects
@@
 		)
 	)
-	(label "3V3"
-		(at 26.67 175.26 0)
+	(label "SENS_3V3"
+		(at 25.4 175.26 0)
 		(effects
 			(font
@@
 		)
 	)
-	(label "3V3"
-		(at 270.51 87.63 180)
+	(label "SENS_3V3"
+		(at 276.86 87.63 180)
 		(effects
 			(font
@@
 			)
 		)
-		(property "Manufacturer Part" ""
+		(property "Manufacturer Part" "CL05B104KP5NNNC"
 			(at 35.56 168.91 0)
 			(effects
@@
 			)
 		)
-		(property "Manufacturer Part" ""
+		(property "Manufacturer Part" "ICM-42688-P"
 			(at 204.47 77.47 0)
 			(effects
@@
 			)
 		)
-		(property "Manufacturer Part" ""
+		(property "Manufacturer Part" "TMP121AIDBVR"
 			(at 125.73 171.45 0)
 			(effects
@@
 			)
 		)
-		(property "Manufacturer Part" ""
+		(property "Manufacturer Part" "CL05B104KP5NNNC"
 			(at 78.74 168.91 0)
 			(effects
@@
 			)
 		)
-		(property "Manufacturer Part" ""
+		(property "Manufacturer Part" "BMP581"
 			(at 36.83 175.26 0)
 			(effects
@@
 			)
 		)
-		(property "Manufacturer Part" ""
+		(property "Manufacturer Part" "CL10X106MO8NRNC"
 			(at 266.7 147.32 0)
 			(effects
@@
 			)
 		)
-		(property "Manufacturer Part" ""
+		(property "Manufacturer Part" "CL05B104KP5NNNC"
 			(at 194.31 91.44 0)
 			(effects
@@
 			)
 		)
+		(property "Manufacturer Part" "TPS22919DCKR"
+			(at 62.23 139.7 0)
+			(effects
+				(font
+					(size 1.27 1.27)
+				)
+				(hide yes)
+			)
+		)
 		(pin "3"
 		)
@@
 			)
 		)
-		(property "Manufacturer Part" ""
+		(property "Manufacturer Part" "CL10B105MO8NNWC"
 			(at 26.67 86.36 0)
 			(effects
@@
 			)
 		)
-		(property "Manufacturer Part" ""
+		(property "Manufacturer Part" "MMC5983MA"
 			(at 209.55 128.27 0)
 			(effects
@@
 			)
 		)
+		(property "Manufacturer Part" "TPS22919DCKR"
+			(at 62.23 90.17 0)
+			(effects
+				(font
+					(size 1.27 1.27)
+				)
+				(hide yes)
+			)
+		)
 		(pin "3"
 		)
@@
 			)
 		)
-		(property "Manufacturer Part" ""
+		(property "Manufacturer Part" "CL10X106MO8NRNC"
 			(at 85.09 88.9 0)
 			(effects
@@
 			)
 		)
-		(property "Manufacturer Part" ""
+		(property "Manufacturer Part" "CL10X106MO8NRNC"
 			(at 85.09 138.43 0)
 			(effects
@@
 			)
 		)
+		(property "Manufacturer Part" "2328702-8"
+			(at 165.1 88.9 0)
+			(effects
+				(font
+					(size 1.27 1.27)
+				)
+				(hide yes)
+			)
+		)
 		(pin "1"
 		)
@@
 			)
 		)
-		(property "Manufacturer Part" ""
+		(property "Manufacturer Part" "CL10B105MO8NNWC"
 			(at 92.71 88.9 0)
 			(effects
@@
 			)
 		)
-		(property "Manufacturer Part" ""
+		(property "Manufacturer Part" "CL10B105MO8NNWC"
 			(at 26.67 135.89 0)
 			(effects
@@
 			)
 		)
-		(property "Manufacturer Part" ""
+		(property "Manufacturer Part" "CL05B104KP5NNNC"
 			(at 125.73 180.34 0)
 			(effects
@@
 			)
 		)
-		(property "Manufacturer Part" ""
+		(property "Manufacturer Part" "1-2328702-0"
 			(at 165.1 133.35 0)
 			(effects
@@
 			)
 		)
-		(property "Manufacturer Part" ""
+		(property "Manufacturer Part" "CL10B105MO8NNWC"
 			(at 92.71 138.43 0)
 			(effects
@@
 			)
 		)
-		(property "Manufacturer Part" ""
+		(property "Manufacturer Part" "CL10B105MO8NNWC"
 			(at 189.23 134.62 0)
 			(effects
@@
 			)
 		)
-		(property "Manufacturer Part" ""
+		(property "Manufacturer Part" "CL05B104KP5NNNC"
 			(at 266.7 96.52 0)
 			(effects
