File: EDA/sub/bottom_asm/bottom_asm.kicad_sch (KiCad schematic)
At the start: 6 parts, among them J1 1-2328702-0, U1 TMP121AIDBVR, U2 VL53L1CXV0FY_1

Commit message: Uploaded work
Parts:
- added R1, R2: 4.7kΩ, Resistor_SMD:R_0402_1005Metric, symbol Device:R
Connections:
- net SCL: now also R1.2
- net SDA: now also R2.2
- net VDD: now also R1.1, R2.1

Commit message: PCB done
Parts:
- C1, C3: Manufacturer Part (none) -> CL05B104KP5NNNC
- C2: Manufacturer Part (none) -> CL10A475KP8NNNC
- J1: Manufacturer Part (none) -> 1-2328702-0
- R1, R2: Manufacturer Part (none) -> RC0402JR-074K7L
- U1: Manufacturer Part (none) -> TMP121AIDBVR
- U2: footprint VL53L1CXV0FY_1:SENSOR_VL53L1CXV0FY_1 -> CANSAT-lib:SENSOR_VL53L1CXV0FY_1; Manufacturer Part (none) -> VL53L1CXV0FY/1
Changed lines of the file:
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@@
+			)
+		)
+		(property "Manufacturer Part" "1-2328702-0"
+			(at 171.45 59.69 0)
+			(effects
+				(font
+					(size 1.27 1.27)
+				)
+				(hide yes)
 			)
 		)
@@
 			)
 		)
-		(property "Footprint" "VL53L1CXV0FY_1:SENSOR_VL53L1CXV0FY_1"
+		(property "Footprint" "CANSAT-lib:SENSOR_VL53L1CXV0FY_1"
 			(at 111.76 106.68 0)
 			(effects
@@
 				)
 				(justify bottom)
+				(hide yes)
+			)
+		)
+		(property "Manufacturer Part" "VL53L1CXV0FY/1"
+			(at 111.76 106.68 0)
+			(effects
+				(font
+					(size 1.27 1.27)
+				)
 				(hide yes)
 			)
@@
 			)
 		)
+		(property "Manufacturer Part" "CL05B104KP5NNNC"
+			(at 93.98 76.2 0)
+			(effects
+				(font
+					(size 1.27 1.27)
+				)
+				(hide yes)
+			)
+		)
 		(pin "1"
 		)
@@
 			)
 		)
+		(property "Manufacturer Part" "TMP121AIDBVR"
+			(at 96.52 67.31 0)
+			(effects
+				(font
+					(size 1.27 1.27)
+				)
+				(hide yes)
+			)
+		)
 		(pin "6"
 		)
@@
 		)
 		(property "Type" ""
+			(at 143.51 100.33 0)
+			(effects
+				(font
+					(size 1.27 1.27)
+				)
+				(hide yes)
+			)
+		)
+		(property "Manufacturer Part" "CL05B104KP5NNNC"
 			(at 143.51 100.33 0)
 			(effects
@@
 			)
 		)
-		(property "Manufacturer Part" ""
+		(property "Manufacturer Part" "RC0402JR-074K7L"
 			(at 130.81 50.8 0)
 			(effects
@@
 		)
 		(property "Type" ""
+			(at 151.13 100.33 0)
+			(effects
+				(font
+					(size 1.27 1.27)
+				)
+				(hide yes)
+			)
+		)
+		(property "Manufacturer Part" "CL10A475KP8NNNC"
 			(at 151.13 100.33 0)
 			(effects
@@
 			)
 		)
-		(property "Manufacturer Part" ""
+		(property "Manufacturer Part" "RC0402JR-074K7L"
 			(at 138.43 50.8 0)
 			(effects
